Commit message: Fix non-convex collision issue and add AGENTS.md

File: urdf_files/l_shape.urdf (robot description, URDF)
Before this commit: robot l_shape_robot, 1 links, 0 joints
Links:
- link l_shape_link: geometry collision mesh filename=l_shape_vhacd.obj scale=1 1 1; visual mesh filename=l_shape.obj scale=1 1 1
